Commit message: Created publisher only from excel data

File: exo_description/urdf/lleap_exo.urdf.xacro (robot description, xacro)
@@ -17,9 +17,9 @@
   <xacro:property name="joint2" value="knee" />   <!-- thigh to shank -->
   <xacro:property name="joint3" value="ankle" />  <!-- shank to foot -->
-  <gravity>true</gravity>
+  <!-- Joint Type should be: fixed || prismatic || floating -->
   <link name="world"/>
-  <joint name="base" type="fixed">  <!-- Type should be fixed || prismatic -->
-    <origin xyz="1 0 1.3342" rpy="0 0 ${pi}" />
-    <limit lower="-10.0" upper="10.0" effort="100.0" velocity="50.0"/>
+  <joint name="base" type="prismatic">
+    <origin xyz="0 0 1.23" rpy="0 0 ${pi}" />    <!-- 1.24 -->
+    <limit lower="-10.0" upper="10.0" effort="100.0" velocity="100.0"/>
     <parent link="world"/>
     <child link="base_link"/>
@@ -142,5 +142,5 @@
       <axis xyz="0 0 1" />
       <!-- Positional joint limits NOT based on Tamar's msts, but normal ranges instead. -->
-      <limit lower="${ankle_lower_radians}" upper="${ankle_upper_radians}" effort="250" velocity="1.308" />
+      <limit lower="-0.1" upper="0.3" effort="250" velocity="1.308"/>
     </joint>
     <!-- link3 should be the foot. -->
@@ -153,5 +153,5 @@
         <origin xyz="0 0.05 0" rpy="${pi / 2} 0 0" />
         <geometry>
-          <box size="0.05 0.1 0.2"/>
+          <box size="0.03 0.1 0.17"/>
         </geometry>
         <material name="red"/>
@@ -160,5 +160,5 @@
         <origin xyz="0 0.05 0" rpy="${pi / 2} 0 0" />
         <geometry>
-          <box size="0.05 0.1 0.2"/>
+          <box size="0.03 0.1 0.17"/>
         </geometry>
       </collision>

Commit message: Updated urdf for dynamic joint params

File: exo_description/urdf/lleap_exo.urdf.xacro (robot description, xacro)
@@ -17,9 +17,8 @@
   <xacro:property name="joint2" value="knee" />   <!-- thigh to shank -->
   <xacro:property name="joint3" value="ankle" />  <!-- shank to foot -->
-  <!-- Joint Type should be: fixed || prismatic || floating -->
   <link name="world"/>
-  <joint name="base" type="prismatic">
-    <origin xyz="0 0 1.23" rpy="0 0 ${pi}" />    <!-- 1.24 -->
-    <limit lower="-10.0" upper="10.0" effort="100.0" velocity="100.0"/>
+  <joint name="base" type="fixed">
+    <origin xyz="0 0 1.214" rpy="0 0 ${pi}" />    <!-- 1.24 -->
+    <!-- <limit lower="-10.0" upper="10.0" effort="100.0" velocity="100.0"/> -->
     <parent link="world"/>
     <child link="base_link"/>
@@ -73,4 +72,5 @@
       <!-- Positional joint limits partially based on joint calculations. -->
       <limit lower="${hip_lower_radians}" upper="${hip_upper_radians}" effort="700" velocity="5" />
+      <dynamics damping="0.3" friction="0.1"/>
     </joint>
     <!-- link1 should be the thigh (joint1 to joint2).
@@ -107,4 +107,5 @@
       <!-- Positional joint limits partially based on Tamar's msts (lower lim here). -->
       <limit lower="${knee_lower_radians}" upper="${knee_upper_radians}" effort="250" velocity="1.308" />
+      <dynamics damping="0.5" friction="0.4"/>
     </joint>
     <!-- link2 should be the shank (joint2 to joint3).
@@ -143,4 +144,5 @@
       <!-- Positional joint limits NOT based on Tamar's msts, but normal ranges instead. -->
       <limit lower="-0.1" upper="0.3" effort="250" velocity="1.308"/>
+      <dynamics damping="0.7" friction="0.5"/>
     </joint>
     <!-- link3 should be the foot. -->

Commit message: Updated for more robust control of GAIT

File: exo_description/urdf/lleap_exo.urdf.xacro (robot description, xacro)
@@ -19,5 +19,5 @@
   <link name="world"/>
   <joint name="base" type="fixed">
-    <origin xyz="0 0 1.214" rpy="0 0 ${pi}" />    <!-- 1.24 -->
+    <origin xyz="0 0 2.214" rpy="0 0 ${pi}" />    <!-- 1.24 -->
     <!-- <limit lower="-10.0" upper="10.0" effort="100.0" velocity="100.0"/> -->
     <parent link="world"/>

Commit message: Added floating robot model and publishing

File: exo_description/urdf/lleap_exo.urdf.xacro (robot description, xacro)
@@ -17,22 +17,88 @@
   <xacro:property name="joint2" value="knee" />   <!-- thigh to shank -->
   <xacro:property name="joint3" value="ankle" />  <!-- shank to foot -->
+  <!-- === Free Robot. No world link. No base joint === -->
+  <!-- <link name="base_link">
+    <inertial>
+      <origin xyz="0 0 0.5" rpy="0 0 0"/>
+      <mass value="1.0"/>
+      <inertia ixx="0.1041667" ixy="0" ixz="0"
+               iyy="0.0885417" iyz="0"
+               izz="0.0260417"/>
+    </inertial>
+    <visual>
+      <origin xyz="0 0 0.5" rpy="0 0 0"/>
+      <geometry><box size="0.25 0.5 1"/></geometry>
+      <material name="red"/>
+    </visual>
+    <collision>
+      <origin xyz="0 0 0.5" rpy="0 0 0"/>
+      <geometry><box size="0.25 0.5 1"/></geometry>
+    </collision>
+  </link>
+  <gazebo reference="base_link">
+    <pose>0 0 1.214 0 0 3.14159</pose>
+  </gazebo> -->
+  <!-- === Allowing X and Z axis only === -->
+  <link name="base_link">
+    <inertial>
+      <origin xyz="0 0 0.5" rpy="0 0 0"/>
+      <mass value="1.0"/>
+      <inertia ixx="0.1041667" ixy="0" ixz="0"
+              iyy="0.0885417" iyz="0"
+              izz="0.0260417"/>
+    </inertial>
+    <visual>
+      <origin xyz="0 0 0.5" rpy="0 0 0"/>
+      <geometry><box size="0.25 0.5 1"/></geometry>
+      <material name="red"/>
+    </visual>
+    <collision>
+      <origin xyz="0 0 0.5" rpy="0 0 0"/>
+      <geometry><box size="0.25 0.5 1"/></geometry>
+    </collision>
+  </link>
   <link name="world"/>
-  <joint name="base" type="fixed">
-    <origin xyz="0 0 2.214" rpy="0 0 ${pi}" />    <!-- 1.24 -->
-    <!-- <limit lower="-10.0" upper="10.0" effort="100.0" velocity="100.0"/> -->
+  <link name="slider_z">
+    <inertial>
+      <origin xyz="0 0 0" rpy="0 0 0"/>
+      <mass value="0.1"/>
+      <inertia ixx="0.0002083" ixy="0" ixz="0"
+              iyy="0.0002083" iyz="0"
+              izz="0.0002083"/>
+    </inertial>
+    <collision><geometry><sphere radius="0.01"/></geometry></collision>
+    <visual><geometry><sphere radius="0.01"/></geometry></visual>
+  </link>
+  <link name="slider_x">
+    <inertial>
+      <origin xyz="0 0 0" rpy="0 0 0"/>
+      <mass value="0.1"/>
+      <inertia ixx="0.0002083" ixy="0" ixz="0"
+              iyy="0.0002083" iyz="0"
+              izz="0.0002083"/>
+    </inertial>
+    <collision><geometry><sphere radius="0.01"/></geometry></collision>
+    <visual><geometry><sphere radius="0.01"/></geometry></visual>
+  </link>
+  <joint name="base_z" type="prismatic">
+    <origin xyz="0 0 1.214" rpy="0 0 ${pi}"/>
     <parent link="world"/>
+    <child link="slider_z"/>
+    <axis xyz="0 0 1"/>
+    <limit lower="-0.5" upper="0.5" effort="500" velocity="1.0"/>
+    <dynamics damping="50.0" friction="1.0"/>
+  </joint>
+  <joint name="base_x" type="prismatic">
+    <origin xyz="0 0 0" rpy="0 0 0"/>
+    <parent link="slider_z"/>
+    <child link="slider_x"/>
+    <axis xyz="1 0 0"/>
+    <limit lower="-5.0" upper="5.0" effort="500" velocity="1.0"/>
+    <dynamics damping="5.0" friction="0.5"/>
+  </joint>
+  <joint name="base_to_body" type="fixed">
+    <parent link="slider_x"/>
     <child link="base_link"/>
   </joint>
-  <!-- torso: base for the model; attached to world in gazebo if whole model fixed -->
-  <link name="base_link">
-    <visual>
-      <origin xyz="0 0 0.5" rpy="0 0 0" />
-      <mass value="1" />
-      <geometry>
-        <box size="0.25 ${torso_width} 1"/>
-      </geometry>
-      <material name="red"/>
-    </visual>
-  </link>
   <xacro:macro name="leg" params="prefix reflect">
     <joint name="${prefix}_${joint0}_fixed_joint" type="fixed">
@@ -136,12 +202,9 @@
     <joint name="${prefix}_${joint3}_revolute_joint" type="revolute">
       <origin xyz="${0.475 + 0.075} 0.003 -0.03" rpy="0 0 0" />
-      <!-- TODO: once make simplified collisional geometries (dimensions based on SolidWorks models > ask design team),
-      use those known dimensions to place the ankle joint origin at the bottom of the shank.
-      Then use similar math (foot box dimensions) to place the foot link origin relative to the ankle joint origin. -->
       <parent link="${prefix}_${link2}" />
       <child link="${prefix}_${link3}" />
       <axis xyz="0 0 1" />
       <!-- Positional joint limits NOT based on Tamar's msts, but normal ranges instead. -->
-      <limit lower="-0.1" upper="0.3" effort="250" velocity="1.308"/>
+      <limit lower="-0.6" upper="0.3" effort="250" velocity="1.308"/>
       <dynamics damping="0.7" friction="0.5"/>
     </joint>
@@ -170,5 +233,4 @@
   <xacro:leg prefix="right" reflect="1" />
   <xacro:leg prefix="left" reflect="-1.75" />
-  <dynamics damping="50.0" friction="50.0"/>
   <!-- All ros2_control needed parameters for interface between Gazebo and ROS -->
   <ros2_control name="exosuit" type="system">

Commit message: Corrected robot urdf (added X - Z free columns)

File: exo_description/urdf/lleap_exo.urdf.xacro (robot description, xacro)
@@ -82,5 +82,5 @@
   </link>
   <joint name="base_z" type="prismatic">
-    <origin xyz="0 0 1.214" rpy="0 0 ${pi}"/>
+    <origin xyz="0 0 1.22" rpy="0 0 ${pi}"/>
     <parent link="world"/>
     <child link="slider_z"/>
@@ -173,5 +173,5 @@
       <!-- Positional joint limits partially based on Tamar's msts (lower lim here). -->
       <limit lower="${knee_lower_radians}" upper="${knee_upper_radians}" effort="250" velocity="1.308" />
-      <dynamics damping="0.5" friction="0.4"/>
+      <dynamics damping="4.0" friction="1.0"/>
     </joint>
     <!-- link2 should be the shank (joint2 to joint3).

Commit message: Updated the scaling from nn and correct urdf model

File: exo_description/urdf/lleap_exo.urdf.xacro (robot description, xacro)
@@ -137,5 +137,5 @@
       <axis xyz="0 0 1" />
       <!-- Positional joint limits partially based on joint calculations. -->
-      <limit lower="${hip_lower_radians}" upper="${hip_upper_radians}" effort="700" velocity="5" />
+      <limit lower="-10.0" upper="10.0"  effort="700" velocity="5" />
       <dynamics damping="0.3" friction="0.1"/>
     </joint>
@@ -172,5 +172,5 @@
       <axis xyz="0 0 1" />
       <!-- Positional joint limits partially based on Tamar's msts (lower lim here). -->
-      <limit lower="${knee_lower_radians}" upper="${knee_upper_radians}" effort="250" velocity="1.308" />
+      <limit lower="-10.0" upper="10.0" effort="250" velocity="1.308" />
       <dynamics damping="4.0" friction="1.0"/>
     </joint>
@@ -206,5 +206,5 @@
       <axis xyz="0 0 1" />
       <!-- Positional joint limits NOT based on Tamar's msts, but normal ranges instead. -->
-      <limit lower="-0.6" upper="0.3" effort="250" velocity="1.308"/>
+      <limit lower="-10.0" upper="10.0"  effort="250" velocity="1.308"/>
       <dynamics damping="0.7" friction="0.5"/>
     </joint>

Commit message: Update on simple publisher and controller gains

File: exo_description/urdf/lleap_exo.urdf.xacro (robot description, xacro)
@@ -82,5 +82,5 @@
   </link>
   <joint name="base_z" type="prismatic">
-    <origin xyz="0 0 1.22" rpy="0 0 ${pi}"/>
+    <origin xyz="0 0 2.22" rpy="0 0 ${pi}"/>
     <parent link="world"/>
     <child link="slider_z"/>
@@ -264,5 +264,5 @@
   </ros2_control>
    <gazebo>  <!-- Gazebo - Ros plugin for (exo_control) controller package to work-->
-    <plugin filename="libign_ros2_control-system.so" name="ign_ros2_control::IgnitionROS2ControlPlugin">
+    <plugin filename="libign_ros2_control-system.so" name="gz_ros2_control::IgnitionROS2ControlPlugin">
       <robot_param>robot_description</robot_param>
       <robot_param_node>robot_state_publisher</robot_param_node>

Commit message: Corrected plugin and update on pd controller

File: exo_description/urdf/lleap_exo.urdf.xacro (robot description, xacro)
@@ -87,5 +87,5 @@
     <axis xyz="0 0 1"/>
     <limit lower="-0.5" upper="0.5" effort="500" velocity="1.0"/>
-    <dynamics damping="50.0" friction="1.0"/>
+    <dynamics damping="5.0" friction="1.0"/>
   </joint>
   <joint name="base_x" type="prismatic">
@@ -173,5 +173,5 @@
       <!-- Positional joint limits partially based on Tamar's msts (lower lim here). -->
       <limit lower="-10.0" upper="10.0" effort="250" velocity="1.308" />
-      <dynamics damping="4.0" friction="1.0"/>
+      <dynamics damping="0.4" friction="1.0"/>
     </joint>
     <!-- link2 should be the shank (joint2 to joint3).
@@ -264,5 +264,5 @@
   </ros2_control>
    <gazebo>  <!-- Gazebo - Ros plugin for (exo_control) controller package to work-->
-    <plugin filename="libign_ros2_control-system.so" name="gz_ros2_control::IgnitionROS2ControlPlugin">
+    <plugin filename="libign_ros2_control-system.so" name="ign_ros2_control::IgnitionROS2ControlPlugin">
       <robot_param>robot_description</robot_param>
       <robot_param_node>robot_state_publisher</robot_param_node>

Commit message: More sane attemts on using kinematics and kinetics for better exoskeleton control

File: exo_description/urdf/lleap_exo.urdf.xacro (robot description, xacro)
@@ -82,5 +82,5 @@
   </link>
   <joint name="base_z" type="prismatic">
-    <origin xyz="0 0 2.22" rpy="0 0 ${pi}"/>
+    <origin xyz="0 0 1.22" rpy="0 0 ${pi}"/>
     <parent link="world"/>
     <child link="slider_z"/>
@@ -233,5 +233,4 @@
   <xacro:leg prefix="right" reflect="1" />
   <xacro:leg prefix="left" reflect="-1.75" />
-  <!-- All ros2_control needed parameters for interface between Gazebo and ROS -->
   <ros2_control name="exosuit" type="system">
     <hardware>
@@ -241,24 +240,36 @@
       <command_interface name="position"/>
       <state_interface name="position"/>
+      <state_interface name="velocity"/>
+      <state_interface name="effort"/>
     </joint>
     <joint name="left_knee_revolute_joint">
       <command_interface name="position"/>
       <state_interface name="position"/>
+      <state_interface name="velocity"/>
+      <state_interface name="effort"/>
     </joint>
     <joint name="left_ankle_revolute_joint">
       <command_interface name="position"/>
       <state_interface name="position"/>
+      <state_interface name="velocity"/>
+      <state_interface name="effort"/>
     </joint>
     <joint name="right_hip_revolute_joint">
       <command_interface name="position"/>
       <state_interface name="position"/>
+      <state_interface name="velocity"/>
+      <state_interface name="effort"/>
     </joint>
     <joint name="right_knee_revolute_joint">
       <command_interface name="position"/>
       <state_interface name="position"/>
+      <state_interface name="velocity"/>
+      <state_interface name="effort"/>
     </joint>
     <joint name="right_ankle_revolute_joint">
       <command_interface name="position"/>
       <state_interface name="position"/>
+      <state_interface name="velocity"/>
+      <state_interface name="effort"/>
     </joint>
   </ros2_control>

Commit message: Update lleap exo model for foot contact sensors

File: exo_description/urdf/lleap_exo.urdf.xacro (robot description, xacro)
@@ -13,30 +13,14 @@
   <xacro:property name="torso_width" value="0.5"/>   <!-- in meters -->
   <!-- repeated leg joint names -->
+  <xacro:property name="width" value="0.05"/>
   <xacro:property name="joint0" value="pelvis" /> <!-- hip base to torso; fixed! -->
   <xacro:property name="joint1" value="hip" />    <!-- fixed to thigh -->
   <xacro:property name="joint2" value="knee" />   <!-- thigh to shank -->
   <xacro:property name="joint3" value="ankle" />  <!-- shank to foot -->
-  <!-- === Free Robot. No world link. No base joint === -->
-  <!-- <link name="base_link">
-    <inertial>
-      <origin xyz="0 0 0.5" rpy="0 0 0"/>
-      <mass value="1.0"/>
-      <inertia ixx="0.1041667" ixy="0" ixz="0"
-               iyy="0.0885417" iyz="0"
-               izz="0.0260417"/>
-    </inertial>
-    <visual>
-      <origin xyz="0 0 0.5" rpy="0 0 0"/>
-      <geometry><box size="0.25 0.5 1"/></geometry>
-      <material name="red"/>
-    </visual>
-    <collision>
-      <origin xyz="0 0 0.5" rpy="0 0 0"/>
-      <geometry><box size="0.25 0.5 1"/></geometry>
-    </collision>
-  </link>
-  <gazebo reference="base_link">
-    <pose>0 0 1.214 0 0 3.14159</pose>
-  </gazebo> -->
+  <xacro:property name="origin_y_thigh" value="0.043454"/>
+  <!-- Foot sole contact -->
+  <xacro:property name="foot_size_y" value="0.10"/>  <!-- width (side-to-side) -->
+  <xacro:property name="foot_size_z" value="0.17"/>  <!-- length (forward) -->
+  <xacro:property name="sole_thick"  value="0.001"/>
   <!-- === Allowing X and Z axis only === -->
   <link name="base_link">
@@ -82,5 +66,5 @@
   </link>
   <joint name="base_z" type="prismatic">
-    <origin xyz="0 0 1.22" rpy="0 0 ${pi}"/>
+    <origin xyz="0 0 1.23" rpy="0 0 ${pi}"/>
     <parent link="world"/>
     <child link="slider_z"/>
@@ -129,7 +113,10 @@
       </collision>
     </link>
+    <xacro:if value="${int(reflect) &lt; 0}">
+      <xacro:property name="origin_y_thigh" value="0.123454"/>
+    </xacro:if>
     <!-- hip joint: fixed hip base to thigh (link1) -->
     <joint name="${prefix}_${joint1}_revolute_joint" type="revolute">
-      <origin xyz="0.00012638 0.043454 -0.0003763" rpy="${pi / 2} ${pi / 2} ${pi}" />
+      <origin xyz="0.00012638 ${origin_y_thigh} -0.0003763" rpy="${pi / 2} ${pi / 2} ${pi}" />
       <parent link="${prefix}_${link0}" />
       <child link="${prefix}_${link1}" />
@@ -229,4 +216,38 @@
       </collision>
     </link>
+    <!-- Extra joint + link for sole contact sensor -->
+    <joint name="${prefix}_foot_to_sole_sensor" type="fixed">
+      <origin xyz="0.015 0.05 0" rpy="0 ${pi/2} 0"/>
+      <parent link="${prefix}_${link3}"/>
+      <child link="${prefix}_sole_sensor"/>
+    </joint>
+    <link name="${prefix}_sole_sensor">
+      <inertial>
+        <origin xyz="0 0 0" rpy="0 0 0"/>
+        <mass value="0.001"/>
+        <inertia ixx="1e-6" ixy="0" ixz="0" iyy="1e-6" iyz="0" izz="1e-6"/></inertial>
+      <visual>
+        <origin xyz="0 0 0" rpy="0 ${pi/2} ${pi/2}"/>
+        <geometry>
+          <box size="${sole_thick} ${foot_size_y} ${foot_size_z}"/>
+        </geometry>
+        <material name="dark_gray"/>
+      </visual>
+      <collision>
+        <origin xyz="0 0 0" rpy="0 ${pi/2} ${pi/2}"/>
+        <geometry>
+          <box size="${sole_thick} ${foot_size_y} ${foot_size_z}"/>
+        </geometry>
+      </collision>
+    </link>
+    <gazebo reference="${prefix}_sole_sensor">
+      <sensor name="${prefix}_sole_contact" type="contact">
+        <always_on>1</always_on>
+        <update_rate>200</update_rate>
+        <contact>
+          <collision>${prefix}_foot_fixed_joint_lump__${prefix}_sole_sensor_collision_1</collision>
+        </contact>
+      </sensor>
+    </gazebo>
   </xacro:macro>
   <!-- Legs actually created. -->

Commit message: PV controller correct training-> publishing order

File: exo_description/urdf/lleap_exo.urdf.xacro (robot description, xacro)
@@ -13,5 +13,4 @@
   <xacro:property name="torso_width" value="0.5"/>   <!-- in meters -->
   <!-- repeated leg joint names -->
-  <xacro:property name="width" value="0.05"/>
   <xacro:property name="joint0" value="pelvis" /> <!-- hip base to torso; fixed! -->
   <xacro:property name="joint1" value="hip" />    <!-- fixed to thigh -->
@@ -78,5 +77,5 @@
     <child link="slider_x"/>
     <axis xyz="1 0 0"/>
-    <limit lower="-5.0" upper="5.0" effort="500" velocity="1.0"/>
+    <limit lower="-5.0" upper="10.0" effort="500" velocity="1.0"/>
     <dynamics damping="5.0" friction="0.5"/>
   </joint>
@@ -159,5 +158,5 @@
       <axis xyz="0 0 1" />
       <!-- Positional joint limits partially based on Tamar's msts (lower lim here). -->
-      <limit lower="-10.0" upper="10.0" effort="250" velocity="1.308" />
+      <limit lower="-10.0" upper="0.0" effort="250" velocity="1.308" />
       <dynamics damping="0.4" friction="1.0"/>
     </joint>
@@ -232,5 +231,5 @@
           <box size="${sole_thick} ${foot_size_y} ${foot_size_z}"/>
         </geometry>
-        <material name="dark_gray"/>
+        <material name="orange"/>
       </visual>
       <collision>
